File: power_supply_1.03.sch (KiCad schematic (older format))
At the start: 74 parts, among them J1 12v, 0.5A nominal, 5A Surge, J10 M1 Disconnect, J2 Power Switch, J3 Shutdown, J4 12V 5V, J5 Program, J6 Serial Debug, J7 REMOVE to PRGM, J8 5V 25W, J9 FRAM I2C, M1 XL4015, M2 U1V11F5, M3 U3V70F5, Q1 BSS806, Q2 BSS806, Q3 SPD18P06PGBTMA1, Q4 BSS806, Q5 BSS806, Q6 SQ3495-EV, Q7 BSS806, U1 MCP9700A, U2 BTS443P, U3 ALD910027, U4 PIC16F1709, U5 MCP111-SOT23, U6 MB85RC1MT, U7 MCP1700-3302E_SOT23

Commit message: Version 1.03 fixes M1, J4, SW footprints. R1 schematic error fixed. Heat sink copper area for U2, D5, D9
Parts:
- J4: footprint Connector_PinHeader_2.54mm:PinHeader_1x03_P2.54mm_Vertical -> Connector_JST:JST_XH_B3B-XH-A_1x03_P2.50mm_Vertical
Changed lines of the file:
@@
 F 0 "J4" V 1850 3000 50  0000 R CNN
 F 1 "12V  5V" V 1950 2900 50  0000 R CNN
-F 2 "Connector_PinHeader_2.54mm:PinHeader_1x03_P2.54mm_Vertical" H 1850 2750 50  0001 C CNN
+F 2 "Connector_JST:JST_XH_B3B-XH-A_1x03_P2.50mm_Vertical" H 1850 2750 50  0001 C CNN
 F 3 "~" H 1850 2750 50  0001 C CNN
 F 4 "https://www.amazon.com/Header-Lystaii-Pin-Connector-Electronic/dp/B06ZZN8L9S" H 1850 2750 50  0001 C CNN "Part#"
